File: Dot Matrix/DotMatrix/DotMatrix.kicad_pcb (KiCad board)
At the start: 2 copper layers, 82 x 74.9 mm, 22 parts, among them J1 Gnd, J2 Red, J3 Green

Commit message: Some cleanups
Parts:
- J1: value Gnd -> Anodes
Routing:
- net Net-(J2-Pin_5): track 63.1 -> 67.2 mm
- net Net-(J2-Pin_6): track 52.1 -> 54.8 mm
- net Net-(J3-Pin_5): track 78.7 -> 81.1 mm
- net Net-(J3-Pin_6): track 65.8 -> 67.5 mm
- net Net-(J3-Pin_7): track 51.2 -> 52.2 mm
- net Net-(J3-Pin_8): track 41.9 -> 42.6 mm
Other:
- board text added: "mHBr"
- board text removed: "Designed By mHBr"
