File: Dot Matrix/DotMatrix/DotMatrix.kicad_sch (KiCad schematic)
At the start: 20 parts, among them J1 Gnd, J2 Red, J3 Green

Commit message: Some cleanups
Parts:
- J1: value Gnd -> Anodes
Changed lines of the file:
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@@
 (kicad_sch
-	(version 20231120)
+	(version 20250114)
 	(generator "eeschema")
-	(generator_version "8.0")
+	(generator_version "9.0")
 	(paper "A4")
 	(wire
@@
 			)
 		)
-		(property "Value" "Gnd"
+		(property "Value" "Anodes"
 			(at 100.965 80.01 0)
 			(effects
@@
 		)
 	)
+	(embedded_fonts no)
 )
